Commit message: Configuracion de los archivos xacro para el desino del robot

File: kuka_kr210/kr210_description/urdf/kr210l150_macro.xacro (robot description, xacro)
@@ -165,5 +165,6 @@
       <child link="${prefix}link_1"/>
       <axis xyz="0 0 1"/>
-      <limit lower="${radians(-185)}" upper="${radians(185)}" effort="0" velocity="${radians(123)}"/>
+      <limit lower="${radians(-185)}" upper="${radians(185)}" effort="692" velocity="${radians(123)}"/>
+      <dynamics damping="0.0" friction="0.0"/>
     </joint>
     <joint name="${prefix}joint_a2" type="revolute">
@@ -172,5 +173,6 @@
       <child link="${prefix}link_2"/>
       <axis xyz="0 1 0"/>
-      <limit lower="${radians(-45)}" upper="${radians(85)}" effort="0" velocity="${radians(115)}"/>
+      <limit lower="${radians(-45)}" upper="${radians(85)}" effort="574" velocity="${radians(115)}"/>
+      <dynamics damping="0.0" friction="0.0"/>
     </joint>
     <joint name="${prefix}joint_a3" type="revolute">
@@ -179,5 +181,6 @@
       <child link="${prefix}link_3"/>
       <axis xyz="0 1 0"/>
-      <limit lower="${radians(-210)}" upper="${radians(65)}" effort="0" velocity="${radians(112)}"/>
+      <limit lower="${radians(-210)}" upper="${radians(65)}" effort="242" velocity="${radians(112)}"/>
+      <dynamics damping="0.0" friction="0.0"/>
     </joint>
     <joint name="${prefix}joint_a4" type="revolute">
@@ -186,5 +189,6 @@
       <child link="${prefix}link_4"/>
       <axis xyz="1 0 0"/>
-      <limit lower="${radians(-350)}" upper="${radians(350)}" effort="0" velocity="${radians(179)}"/>
+      <limit lower="${radians(-350)}" upper="${radians(350)}" effort="58" velocity="${radians(179)}"/>
+      <dynamics damping="0.0" friction="0.0"/>
     </joint>
     <joint name="${prefix}joint_a5" type="revolute">
@@ -193,5 +197,6 @@
       <child link="${prefix}link_5"/>
       <axis xyz="0 1 0"/>
-      <limit lower="${radians(-125)}" upper="${radians(125)}" effort="0" velocity="${radians(172)}"/>
+      <limit lower="${radians(-125)}" upper="${radians(125)}" effort="29" velocity="${radians(172)}"/>
+      <dynamics damping="0.0" friction="0.0"/>
     </joint>
     <joint name="${prefix}joint_a6" type="revolute">
@@ -200,5 +205,6 @@
       <child link="${prefix}link_6"/>
       <axis xyz="1 0 0"/>
-      <limit lower="${radians(-350)}" upper="${radians(350)}" effort="0" velocity="${radians(219)}"/>
+      <limit lower="${radians(-350)}" upper="${radians(350)}" effort="29" velocity="${radians(219)}"/>
+      <dynamics damping="0.0" friction="0.0"/>
     </joint>
     <joint name="${prefix}link_6-flange" type="fixed">
