Commit message: Cambio de posicion del gripper

File: kuka_kr210/kr210_gazebo/urdf/gazebo_2f.xacro (robot description, xacro)
@@ -6,5 +6,5 @@
     <parent link="tool0"/>
     <child link="coupling_link"/>
-    <origin rpy="0 0 0" xyz="0 0 -0.003"/>
+    <origin rpy="0 0 0" xyz="0 0 0.01"/>
   </joint>
   <xacro:include filename="$(find kr210_gazebo)/urdf/transmission_2f.xacro"/>
