Commit message: Cambio de dimension y estructura de objetos en la banda

File: kuka_kr210/kr210_gazebo/urdf/blue_cube.urdf (robot description, URDF)
Before this commit: robot blue_cube, 1 links, 0 joints
Links:
- link base_link: geometry collision box size=0.4 0.07 0.2; visual box size=0.4 0.07 0.2

File: kuka_kr210/kr210_gazebo/urdf/green_cube.urdf (robot description, URDF)
Before this commit: robot green_cube, 1 links, 0 joints
Links:
- link base_link: geometry collision box size=0.4 0.07 0.2; visual box size=0.4 0.07 0.2

File: kuka_kr210/kr210_gazebo/urdf/kr210_main.xacro (robot description, xacro)
@@ -5,5 +5,4 @@
     <xacro:arg name="camera_arm" default="false"/>
     <xacro:include filename="$(find kr210_gazebo)/urdf/conveyor.xacro"/>
-    <xacro:include filename="$(find kr210_gazebo)/urdf/box.xacro"/>
     <xacro:include filename="$(find kr210_gazebo)/urdf/gazebo.xacro"/>
     <!-- camera -->

File: kuka_kr210/kr210_gazebo/urdf/red_cube.urdf (robot description, URDF)
Before this commit: robot red_cube, 1 links, 0 joints
Links:
- link base_link: geometry collision box size=0.4 0.07 0.2; visual box size=0.4 0.07 0.2

File: kuka_kr210/kr210_gazebo/urdf/transmission_2f.xacro (robot description, xacro)
@@ -88,5 +88,5 @@
         <plugin filename="libgazebo_grasp_fix.so" name="gazebo_grasp_fix">
         <arm>
-            <arm_name>kuka_kr210</arm_name>
+            <arm_name>kr210</arm_name>
             <palm_link>link_6</palm_link>
             <gripper_link>left_outer_knuckle</gripper_link>

Commit message: Edicion de masa e inercias de las cajas

File: kuka_kr210/kr210_gazebo/urdf/blue_cube.urdf (robot description, URDF)
Before this commit: robot blue_cube, 1 links, 0 joints
Links:
- link base_link: mass 0.1 -> 50.0

File: kuka_kr210/kr210_gazebo/urdf/green_cube.urdf (robot description, URDF)
Before this commit: robot green_cube, 1 links, 0 joints
Links:
- link base_link: mass 0.1 -> 50.0
