Commit message: Actualizacion nombres de las cajas

File: kuka_kr210/kr210_gazebo/urdf/box_blue.urdf (robot description, URDF)
Before this commit: robot red_cube, 1 links, 0 joints
Links:
- link base_link: mass 0.1 -> 50.0

File: kuka_kr210/kr210_gazebo/urdf/box_red.urdf (robot description, URDF)
Before this commit: robot blue_cube, 1 links, 0 joints
Links:
- link base_link: mass 50.0 -> 0.1
