Commit message: Implementacion de camara para vision por computador

File: kuka_kr210/kr210_gazebo/urdf/camera.xacro (robot description, xacro)
@@ -3,21 +3,21 @@
     <link name="camera">
         <collision>
-        <origin rpy="0 0 0" xyz="0 0 0"/>
-        <geometry>
-            <box size="0.1 0.7 0.7"/>
-        </geometry>
+            <origin rpy="0 0 0" xyz="0 0 0"/>
+            <geometry>
+                <box size="0.1 0.7 0.7"/>
+            </geometry>
         </collision>
         <visual>
-        <origin rpy="0 0 0" xyz="0 0 0"/>
-        <geometry>
-            <box size="0.1 0.7 0.7"/>
-        </geometry>
-        <material name="grey"/>
+            <origin rpy="0 0 0" xyz="0 0 0"/>
+            <geometry>
+                <box size="0.1 0.7 0.7"/>
+            </geometry>
+            <material name="grey"/>
         </visual>
         <inertial>
-        <mass value="0.1"/>
-        <origin rpy="0 0 0" xyz="0 0 0"/>
-        <box_inertia m="0.1" x="0.1" y="0.7" z="0.7"/>
-        <inertia ixx="1e-6" ixy="0" ixz="0" iyy="1e-6" iyz="0" izz="1e-6"/>
+            <mass value="0.1"/>
+            <origin rpy="0 0 0" xyz="0 0 0"/>
+            <box_inertia m="0.1" x="0.1" y="0.7" z="0.7"/>
+            <inertia ixx="1e-6" ixy="0" ixz="0" iyy="1e-6" iyz="0" izz="1e-6"/>
         </inertial>
     </link>
@@ -30,49 +30,31 @@
     <joint name="camera_joint" type="fixed">
         <axis xyz="0 0 0"/>
-        <origin rpy="0 1.5708 0" xyz="0.5 0 4.5"/>
+        <origin rpy="0 1.5708 0" xyz="0.0 -2.5 3.5"/>
         <parent link="base_link"/>
         <child link="camera"/>
     </joint>
     <gazebo reference="camera">
-        <sensor name="camera1" type="depth">
-        <update_rate>20</update_rate>
-        <camera>
-            <horizontal_fov>1.2</horizontal_fov>
-            <image>
-            <width>640</width>
-            <!--640-->
-            <height>480</height>
-            <!--480-->
-            <format>R8G8B8</format>
-            </image>
-            <clip>
-            <near>0.05</near>
-            <far>30</far>
-            </clip>
-        </camera>
-        <plugin filename="libgazebo_ros_openni_kinect.so" name="camera_controller">
-            <baseline>0.2</baseline>
-            <alwaysOn>false</alwaysOn>
-            <updateRate>1.0</updateRate>
-            <cameraName>camera1</cameraName>
-            <imageTopicName>/camera1/color/image_raw</imageTopicName>
-            <cameraInfoTopicName>/camera1/color/camera_info</cameraInfoTopicName>
-            <depthImageTopicName>/camera1/depth/image_raw</depthImageTopicName>
-            <depthImageInfoTopicName>/camera1/depth/camera_info</depthImageInfoTopicName>
-            <pointCloudTopicName>/camera1/depth/points</pointCloudTopicName>
-            <frameName>camera_frame_optical</frameName>
-            <pointCloudCutoff>0.5</pointCloudCutoff>
-            <pointCloudCutoffMax>3.0</pointCloudCutoffMax>
-            <distortionK1>0.00000001</distortionK1>
-            <distortionK2>0.00000001</distortionK2>
-            <distortionK3>0.00000001</distortionK3>
-            <distortionT1>0.00000001</distortionT1>
-            <distortionT2>0.00000001</distortionT2>
-            <CxPrime>0</CxPrime>
-            <Cx>0</Cx>
-            <Cy>0</Cy>
-            <focalLength>0</focalLength>
-            <hackBaseline>0</hackBaseline>
-        </plugin>
+        <sensor name="camera1" type="camera">
+            <update_rate>20</update_rate>
+            <camera>
+                <horizontal_fov>1.2</horizontal_fov>
+                <image>
+                    <width>640</width>
+                    <height>480</height>
+                    <format>R8G8B8</format>
+                </image>
+                <clip>
+                    <near>0.05</near>
+                    <far>30</far>
+                </clip>
+            </camera>
+            <plugin filename="libgazebo_ros_camera.so" name="camera_controller">
+                <alwaysOn>true</alwaysOn>
+                <updateRate>20.0</updateRate>
+                <cameraName>camera1</cameraName>
+                <imageTopicName>/camera1/image_raw</imageTopicName>
+                <cameraInfoTopicName>/camera1/camera_info</cameraInfoTopicName>
+                <frameName>camera_frame_optical</frameName>
+            </plugin>
         </sensor>
     </gazebo>

Commit message: Actualizacion de xacro de la camara

File: kuka_kr210/kr210_gazebo/urdf/camera.xacro (robot description, xacro)
@@ -15,10 +15,7 @@
             <material name="grey"/>
         </visual>
-        <inertial>
-            <mass value="0.1"/>
-            <origin rpy="0 0 0" xyz="0 0 0"/>
-            <box_inertia m="0.1" x="0.1" y="0.7" z="0.7"/>
-            <inertia ixx="1e-6" ixy="0" ixz="0" iyy="1e-6" iyz="0" izz="1e-6"/>
-        </inertial>
+        <xacro:inertial_box mass="0.1" x="0.1" y="0.7" z="0.7">
+            <origin xyz="0 0 0" rpy="0 0 0"/>
+        </xacro:inertial_box>
     </link>
     <joint name="camera_optical_joint" type="fixed">
@@ -35,4 +32,5 @@
     </joint>
     <gazebo reference="camera">
+        <material>Gazebo/Grey</material>
         <sensor name="camera1" type="camera">
             <update_rate>20</update_rate>
