Commit message: Implementacion del movimiento de la banda con sus respectivas jabas

File: kuka_kr210/kr210_gazebo/urdf/conveyor.xacro (robot description, xacro)
@@ -15,5 +15,5 @@
             <origin xyz="0 0 0" rpy="0 0 0" />
             <geometry>
-                <mesh filename="package://kr210_description/meshes/conveyor/conveyor_belt.stl" scale="1 2 1"/>
+                <mesh filename="package://kr210_description/meshes/conveyor/conveyor_belt.stl" scale="2 2 1"/>
             </geometry>
             <material name="white">
@@ -24,5 +24,5 @@
             <origin xyz="0 0 0" rpy="0 0 0" />
             <geometry>
-                <mesh filename="package://kr210_description/meshes/conveyor/conveyor_belt.stl" scale="1 2 1"/>
+                <mesh filename="package://kr210_description/meshes/conveyor/conveyor_belt.stl" scale="2 2 1"/>
             </geometry>
         </collision>
@@ -41,8 +41,8 @@
             <inertia ixx="0.0" ixy="0.0" ixz="0.0" iyy="0.0" iyz="0.0" izz="0.0"/>
         </inertial>
-         <visual>
+        <visual>
             <origin xyz="0.0 0.0 0.0005" rpy="0.0 0.0 0.0"/>
             <geometry>
-                <box size="0.425 2.4 0.001"/>
+                <box size="0.85 2.4 0.001"/>
             </geometry>
             <material name="test">
@@ -53,5 +53,5 @@
             <origin xyz="0.0 0.0 0.0005" rpy="0.0 0.0 0.0"/>
             <geometry>
-                <box size="0.425 2.4 0.001"/>
+                <box size="0.85 2.4 0.001"/>
             </geometry>
         </collision>

Commit message: Recursos al mundo del piso y paredes para Rviz y Gazebo

File: kuka_kr210/kr210_gazebo/urdf/conveyor.xacro (robot description, xacro)
@@ -17,7 +17,5 @@
                 <mesh filename="package://kr210_description/meshes/conveyor/conveyor_belt.stl" scale="2 2 1"/>
             </geometry>
-            <material name="white">
-                <color rgba="1 1 1 1" />
-            </material>
+            <material name="grey"/>
         </visual>
         <collision>
@@ -65,3 +63,6 @@
         </plugin>
     </gazebo>
+    <gazebo reference="belt_visual">
+        <material>Gazebo/Gray</material>
+    </gazebo>
 </robot>

File: kuka_kr210/kr210_gazebo/urdf/kr210_main.xacro (robot description, xacro)
@@ -5,4 +5,6 @@
     <xacro:include filename="$(find kr210_gazebo)/urdf/resources/inertial_macros.xacro"/>
     <xacro:include filename="$(find kr210_gazebo)/urdf/resources/materials.xacro"/>
+    <xacro:include filename="$(find kr210_gazebo)/urdf/resources/floor.xacro"/>
+    <xacro:include filename="$(find kr210_gazebo)/urdf/resources/wall.xacro"/>
     <xacro:include filename="$(find kr210_gazebo)/urdf/conveyor.xacro"/>
     <xacro:include filename="$(find kr210_gazebo)/urdf/gazebo.xacro"/>

File: kuka_kr210/kr210_gazebo/urdf/resources/materials.xacro (robot description, xacro)
@@ -4,6 +4,12 @@
         <color rgba="0 0 0 1"/>
     </material>
+    <material name="light_black">
+        <color rgba="0.25 0.25 0.25 1"/>
+    </material>
     <material name="grey">
         <color rgba="0.5 0.5 0.5 1"/>
+    </material>
+    <material name="light_grey">
+        <color rgba="0.75 0.75 0.75 1"/>
     </material>
     <material name="white">
