Commit message: Correcion de masa de caja roja y ocultar banda

File: kuka_kr210/kr210_gazebo/urdf/boxes/box_red.urdf (robot description, URDF)
Before this commit: robot box_red, 1 links, 0 joints
Links:
- link base_link: mass 0.1 -> 50.0

File: kuka_kr210/kr210_gazebo/urdf/conveyor.xacro (robot description, xacro)
@@ -41,5 +41,5 @@
             <inertia ixx="0.0" ixy="0.0" ixz="0.0" iyy="0.0" iyz="0.0" izz="0.0"/>
         </inertial>
-        <visual>
+        <!-- <visual>
             <origin xyz="0.0 0.0 0.0005" rpy="0.0 0.0 0.0"/>
             <geometry>
@@ -49,5 +49,5 @@
                 <color rgba="1 0 1 1" />
             </material>
-        </visual>
+        </visual> -->
         <collision>
             <origin xyz="0.0 0.0 0.0005" rpy="0.0 0.0 0.0"/>
