Commit message: Correcion de la masa de las 3 cajas

File: kuka_kr210/kr210_gazebo/urdf/boxes/box_blue.urdf (robot description, URDF)
Before this commit: robot box_blue, 1 links, 0 joints
Links:
- link base_link: mass 50.0 -> 5.0

File: kuka_kr210/kr210_gazebo/urdf/boxes/box_green.urdf (robot description, URDF)
Before this commit: robot box_green, 1 links, 0 joints
Links:
- link base_link: mass 50.0 -> 5.0

File: kuka_kr210/kr210_gazebo/urdf/boxes/box_red.urdf (robot description, URDF)
Before this commit: robot box_red, 1 links, 0 joints
Links:
- link base_link: mass 50.0 -> 5.0
